Commit message: Working 16-point vertical descent sweep, cleaned repo

File: custom_description/ur_gz_with_tip.urdf.xacro (robot description, xacro)
@@ -82,8 +82,4 @@
       <geometry><box size="0.010 0.015 0.09"/></geometry>
     </visual>
-    <collision>
-      <origin xyz="0 0 0.03" rpy="0 0 0"/>
-      <geometry><box size="0.010 0.015 0.09"/></geometry>
-    </collision>
     <inertial>
       <mass value="0.02"/>
@@ -101,8 +97,4 @@
       <geometry><box size="0.010 0.015 0.09"/></geometry>
     </visual>
-    <collision>
-      <origin xyz="0 0 0.03" rpy="0 0 0"/>
-      <geometry><box size="0.010 0.015 0.09"/></geometry>
-    </collision>
     <inertial>
       <mass value="0.02"/>
@@ -115,3 +107,9 @@
     <origin xyz="0.008 0 0" rpy="0 0 0"/>
   </joint>
+  <link name="probe_contact_point"/>
+  <joint name="probe_contact_point_joint" type="fixed">
+    <parent link="tool0"/>
+    <child link="probe_contact_point"/>
+    <origin xyz="0 0 0.09" rpy="0 0 0"/>
+  </joint>
 </robot>
